File: PCB/ui.sch (EAGLE design)
At the start: 29 parts

Commit message: UI PCB finished and slickscreen checked
Parts:
- added R8, R9: (no value), rcl:R-EU_R0603
- renumbered RN1 to R10, RN2 to R12, RN3 to R14, RN4 to R11, RN5 to R13, RN6 to R15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
Connections:
- new net SYNC: IC3.SYNC/MODE, IC4.SYNC/MODE, J1.8, R8.1, R9.2
- net +3V3: now also R8.2
- net GND: now also R9.1
